Commit message: Got latest STL files fromNoah

File: waybionic_description/urdf/waybionic.urdf (robot description, URDF)
Before this commit: robot waybionic_placeholder, 2 links, 1 joints
Links:
- removed link arm_link
- added link baseToShoulder_01; collision mesh filename=package://waybionic_description/meshes/baseToShoulder-newDi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 scale=0.001 0.001 0.001; visual mesh filename=package://waybionic_description/meshes/baseToShoulder-newDi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 scale=0.001 0.001 0.001
- added link baseToShoulder_02; collision mesh filename=package://waybionic_description/meshes/baseToShoulder-newDi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 scale=0.001 0.001 0.001; visual mesh filename=package://waybionic_description/meshes/baseToShoulder-newDi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 scale=0.001 0.001 0.001
- added link baseToShoulder_03; collision mesh filename=package://waybionic_description/meshes/baseToShoulder-newDi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 scale=0.001 0.001 0.001; visual mesh filename=package://waybionic_description/meshes/baseToShoulder-newDi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 scale=0.001 0.001 0.001
- added link baseToShoulder_04; collision mesh filename=package://waybionic_description/meshes/baseToShoulder-newDi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 scale=0.001 0.001 0.001; visual mesh filename=package://waybionic_description/meshes/baseToShoulder-newDi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 scale=0.001 0.001 0.001
- added link baseToShoulder_05; collision mesh filename=package://waybionic_description/meshes/baseToShoulder-newDi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 scale=0.001 0.001 0.001; visual mesh filename=package://waybionic_description/meshes/baseToShoulder-newDi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 scale=0.001 0.001 0.001
- added link baseToShoulder_06; collision mesh filename=package://waybionic_description/meshes/baseToShoulder-newDi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 scale=0.001 0.001 0.001; visual mesh filename=package://waybionic_description/meshes/baseToShoulder-newDi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 scale=0.001 0.001 0.001
- added link baseToShoulder_07; collision mesh filename=package://waybionic_description/meshes/baseToShoulder-newDi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 scale=0.001 0.001 0.001; visual mesh filename=package://waybionic_description/meshes/baseToShoulder-newDi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 scale=0.001 0.001 0.001
- added link baseToShoulder_08; collision mesh filename=package://waybionic_description/meshes/baseToShoulder-newDi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 scale=0.001 0.001 0.001; visual mesh filename=package://waybionic_description/meshes/baseToShoulder-newDi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 scale=0.001 0.001 0.001
- added link baseToShoulder_09; collision mesh filename=package://waybionic_description/meshes/baseToShoulder-newDi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 scale=0.001 0.001 0.001; visual mesh filename=package://waybionic_description/meshes/baseToShoulder-newDi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 scale=0.001 0.001 0.001
- added link baseToShoulder_10; collision mesh filename=package://waybionic_description/meshes/baseToShoulder-newDi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 scale=0.001 0.001 0.001; visual mesh filename=package://waybionic_description/meshes/baseToShoulder-newDi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 scale=0.001 0.001 0.001
- added link baseToShoulder_11; collision mesh filename=package://waybionic_description/meshes/baseToShoulder-newDi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 scale=0.001 0.001 0.001; visual mesh filename=package://waybionic_description/meshes/baseToShoulder-newDi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 scale=0.001 0.001 0.001
- added link baseToShoulder_12; collision mesh filename=package://waybionic_description/meshes/baseToShoulder-newDi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 scale=0.001 0.001 0.001; visual mesh filename=package://waybionic_description/meshes/baseToShoulder-newDi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 scale=0.001 0.001 0.001
- added link baseToShoulder_13; collision mesh filename=package://waybionic_description/meshes/baseToShoulder-newDi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 scale=0.001 0.001 0.001; visual mesh filename=package://waybionic_description/meshes/baseToShoulder-newDi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 scale=0.001 0.001 0.001
- added link baseToShoulder_14; collision mesh filename=package://waybionic_description/meshes/baseToShoulder-newDi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 scale=0.001 0.001 0.001; visual mesh filename=package://waybionic_description/meshes/baseToShoulder-newDi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 scale=0.001 0.001 0.001
- added link baseToShoulder_15; collision mesh filename=package://waybionic_description/meshes/baseToShoulder-newDi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 scale=0.001 0.001 0.001; visual mesh filename=package://waybionic_description/meshes/baseToShoulder-newDi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 scale=0.001 0.001 0.001
- added link baseToShoulder_16; collision mesh filename=package://waybionic_description/meshes/baseToShoulder-newDi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 scale=0.001 0.001 0.001; visual mesh filename=package://waybionic_description/meshes/baseToShoulder-newDi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 scale=0.001 0.001 0.001
- added link baseToShoulder_17; collision mesh filename=package://waybionic_description/meshes/baseToShoulder-newDi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 scale=0.001 0.001 0.001; visual mesh filename=package://waybionic_description/meshes/baseToShoulder-newDi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 scale=0.001 0.001 0.001
- added link baseToShoulder_18; collision mesh filename=package://waybionic_description/meshes/baseToShoulder-newDi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 scale=0.001 0.001 0.001; visual mesh filename=package://waybionic_description/meshes/baseToShoulder-newDi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 scale=0.001 0.001 0.001
- added link baseToShoulder_19; collision mesh filename=package://waybionic_description/meshes/baseToShoulder-newDi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 scale=0.001 0.001 0.001; visual mesh filename=package://waybionic_description/meshes/baseToShoulder-newDi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 scale=0.001 0.001 0.001
- added link baseToShoulder_20; collision mesh filename=package://waybionic_description/meshes/baseToShoulder-newDi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 scale=0.001 0.001 0.001; visual mesh filename=package://waybionic_description/meshes/baseToShoulder-newDi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 scale=0.001 0.001 0.001
- added link baseToShoulder_21; collision mesh filename=package://waybionic_description/meshes/baseToShoulder-newDi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 scale=0.001 0.001 0.001; visual mesh filename=package://waybionic_description/meshes/baseToShoulder-newDi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 scale=0.001 0.001 0.001
- added link baseToShoulder_22; collision mesh filename=package://waybionic_description/meshes/baseToShoulder-newDi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 scale=0.001 0.001 0.001; visual mesh filename=package://waybionic_description/meshes/baseToShoulder-newDi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 scale=0.001 0.001 0.001
- added link baseToShoulder_23; collision mesh filename=package://waybionic_description/meshes/baseToShoulder-newDi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 scale=0.001 0.001 0.001; visual mesh filename=package://waybionic_description/meshes/baseToShoulder-newDi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 scale=0.001 0.001 0.001
- added link baseToShoulder_24; collision mesh filename=package://waybionic_description/meshes/baseToShoulder-newDi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 scale=0.001 0.001 0.001; visual mesh filename=package://waybionic_description/meshes/baseToShoulder-newDi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 scale=0.001 0.001 0.001
- added link baseToShoulder_25; collision mesh filename=package://waybionic_description/meshes/baseToShoulder-newDi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 scale=0.001 0.001 0.001; visual mesh filename=package://waybionic_description/meshes/baseToShoulder-newDi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 scale=0.001 0.001 0.001
- added link baseToShoulder_26; collision mesh filename=package://waybionic_description/meshes/baseToShoulder-newDi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 scale=0.001 0.001 0.001; visual mesh filename=package://waybionic_description/meshes/baseToShoulder-newDi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 scale=0.001 0.001 0.001
- added link baseToShoulder_27; collision mesh filename=package://waybionic_description/meshes/baseToShoulder-newDi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 scale=0.001 0.001 0.001; visual mesh filename=package://waybionic_description/meshes/baseToShoulder-newDi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 scale=0.001 0.001 0.001
- added link baseToShoulder_28; collision mesh filename=package://waybionic_description/meshes/baseToShoulder-newDi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 scale=0.001 0.001 0.001; visual mesh filename=package://waybionic_description/meshes/baseToShoulder-newDi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 scale=0.001 0.001 0.001
- added link baseToShoulder_29; collision mesh filename=package://waybionic_description/meshes/baseToShoulder-newDi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 scale=0.001 0.001 0.001; visual mesh filename=package://waybionic_description/meshes/baseToShoulder-newDi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 scale=0.001 0.001 0.001
- added link baseToShoulder_30; collision mesh filename=package://waybionic_description/meshes/baseToShoulder-newDi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 scale=0.001 0.001 0.001; visual mesh filename=package://waybionic_description/meshes/baseToShoulder-newDi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 scale=0.001 0.001 0.001
- added link baseToShoulder_31; collision mesh filename=package://waybionic_description/meshes/baseToShoulder-newDi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 scale=0.001 0.001 0.001; visual mesh filename=package://waybionic_description/meshes/baseToShoulder-newDi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 scale=0.001 0.001 0.001
- added link baseToShoulder_32; collision mesh filename=package://waybionic_description/meshes/baseToShoulder-newDi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 scale=0.001 0.001 0.001; visual mesh filename=package://waybionic_description/meshes/baseToShoulder-newDi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 scale=0.001 0.001 0.001
- added link carrier_to_pulley_01; collision mesh filename=package://waybionic_description/meshes/carrier_to_pulley_fe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 scale=0.001 0.001 0.001; visual mesh filename=package://waybionic_description/meshes/carrier_to_pulley_fe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 scale=0.001 0.001 0.001
- added link carrier_to_pulley_02; collision mesh filename=package://waybionic_description/meshes/carrier_to_pulley_fe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 scale=0.001 0.001 0.001; visual mesh filename=package://waybionic_description/meshes/carrier_to_pulley_fe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 scale=0.001 0.001 0.001
- added link carrier_to_pulley_03; collision mesh filename=package://waybionic_description/meshes/carrier_to_pulley_fe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 scale=0.001 0.001 0.001; visual mesh filename=package://waybionic_description/meshes/carrier_to_pulley_fe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 scale=0.001 0.001 0.001
- added link carrier_to_pulley_04; collision mesh filename=package://waybionic_description/meshes/carrier_to_pulley_fe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 scale=0.001 0.001 0.001; visual mesh filename=package://waybionic_description/meshes/carrier_to_pulley_fe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 scale=0.001 0.001 0.001
- added link carrier_to_pulley_05; collision mesh filename=package://waybionic_description/meshes/carrier_to_pulley_fe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 scale=0.001 0.001 0.001; visual mesh filename=package://waybionic_description/meshes/carrier_to_pulley_fe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 scale=0.001 0.001 0.001
- added link full_arm_jun13_elbow; collision mesh filename=package://waybionic_description/meshes/full-arm-jun13-stl_-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 scale=0.001 0.001 0.001; visual mesh filename=package://waybionic_description/meshes/full-arm-jun13-stl_-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 scale=0.001 0.001 0.001
- added link key_to_diff_01; collision mesh filename=package://waybionic_description/meshes/key-to-diff-mar24-st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 scale=0.001 0.001 0.001; visual mesh filename=package://waybionic_description/meshes/key-to-diff-mar24-st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 scale=0.001 0.001 0.001
- added link key_to_diff_02; collision mesh filename=package://waybionic_description/meshes/key-to-diff-mar24-st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 scale=0.001 0.001 0.001; visual mesh filename=package://waybionic_description/meshes/key-to-diff-mar24-st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 scale=0.001 0.001 0.001
- added link key_to_diff_03; collision mesh filename=package://waybionic_description/meshes/key-to-diff-mar24-st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 scale=0.001 0.001 0.001; visual mesh filename=package://waybionic_description/meshes/key-to-diff-mar24-st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 scale=0.001 0.001 0.001
- added link key_to_diff_04; collision mesh filename=package://waybionic_description/meshes/key-to-diff-mar24-st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 scale=0.001 0.001 0.001; visual mesh filename=package://waybionic_description/meshes/key-to-diff-mar24-st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 scale=0.001 0.001 0.001
- added link key_to_diff_05; collision mesh filename=package://waybionic_description/meshes/key-to-diff-mar24-st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 scale=0.001 0.001 0.001; visual mesh filename=package://waybionic_description/meshes/key-to-diff-mar24-st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 scale=0.001 0.001 0.001
- added link key_to_diff_06; collision mesh filename=package://waybionic_description/meshes/key-to-diff-mar24-st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 scale=0.001 0.001 0.001; visual mesh filename=package://waybionic_description/meshes/key-to-diff-mar24-st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 scale=0.001 0.001 0.001
- added link key_to_diff_07; collision mesh filename=package://waybionic_description/meshes/key-to-diff-mar24-st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 scale=0.001 0.001 0.001; visual mesh filename=package://waybionic_description/meshes/key-to-diff-mar24-st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 scale=0.001 0.001 0.001
- added link key_to_diff_08; collision mesh filename=package://waybionic_description/meshes/key-to-diff-mar24-st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 scale=0.001 0.001 0.001; visual mesh filename=package://waybionic_description/meshes/key-to-diff-mar24-st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 scale=0.001 0.001 0.001
- added link key_to_diff_09; collision mesh filename=package://waybionic_description/meshes/key-to-diff-mar24-st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 scale=0.001 0.001 0.001; visual mesh filename=package://waybionic_description/meshes/key-to-diff-mar24-st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 scale=0.001 0.001 0.001
- added link key_to_diff_10; collision mesh filename=package://waybionic_description/meshes/key-to-diff-mar24-st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 scale=0.001 0.001 0.001; visual mesh filename=package://waybionic_description/meshes/key-to-diff-mar24-st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 scale=0.001 0.001 0.001
- added link key_to_diff_11; collision mesh filename=package://waybionic_description/meshes/key-to-diff-mar24-st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 scale=0.001 0.001 0.001; visual mesh filename=package://waybionic_description/meshes/key-to-diff-mar24-st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 scale=0.001 0.001 0.001
- added link key_to_diff_12; collision mesh filename=package://waybionic_description/meshes/key-to-diff-mar24-st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 scale=0.001 0.001 0.001; visual mesh filename=package://waybionic_description/meshes/key-to-diff-mar24-st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 scale=0.001 0.001 0.001
- added link world
- link base_link: geometry 
Joints:
- removed joint base_to_arm
- added joint j_baseToShoulder_01: type fixed, parent base_link, child baseToShoulder_01, origin xyz=0 0 0 rpy=0 0 0
- added joint j_baseToShoulder_02: type fixed, parent base_link, child baseToShoulder_02, origin xyz=0 0 0 rpy=0 0 0
- added joint j_baseToShoulder_03: type fixed, parent base_link, child baseToShoulder_03, origin xyz=0 0 0 rpy=0 0 0
- added joint j_baseToShoulder_04: type fixed, parent base_link, child baseToShoulder_04, origin xyz=0 0 0 rpy=0 0 0
- added joint j_baseToShoulder_05: type fixed, parent base_link, child baseToShoulder_05, origin xyz=0 0 0 rpy=0 0 0
- added joint j_baseToShoulder_06: type fixed, parent base_link, child baseToShoulder_06, origin xyz=0 0 0 rpy=0 0 0
- added joint j_baseToShoulder_07: type fixed, parent base_link, child baseToShoulder_07, origin xyz=0 0 0 rpy=0 0 0
- added joint j_baseToShoulder_08: type fixed, parent base_link, child baseToShoulder_08, origin xyz=0 0 0 rpy=0 0 0
- added joint j_baseToShoulder_09: type fixed, parent base_link, child baseToShoulder_09, origin xyz=0 0 0 rpy=0 0 0
- added joint j_baseToShoulder_10: type fixed, parent base_link, child baseToShoulder_10, origin xyz=0 0 0 rpy=0 0 0
- added joint j_baseToShoulder_11: type fixed, parent base_link, child baseToShoulder_11, origin xyz=0 0 0 rpy=0 0 0
- added joint j_baseToShoulder_12: type fixed, parent base_link, child baseToShoulder_12, origin xyz=0 0 0 rpy=0 0 0
- added joint j_baseToShoulder_13: type fixed, parent base_link, child baseToShoulder_13, origin xyz=0 0 0 rpy=0 0 0
- added joint j_baseToShoulder_14: type fixed, parent base_link, child baseToShoulder_14, origin xyz=0 0 0 rpy=0 0 0
- added joint j_baseToShoulder_15: type fixed, parent base_link, child baseToShoulder_15, origin xyz=0 0 0 rpy=0 0 0
- added joint j_baseToShoulder_16: type fixed, parent base_link, child baseToShoulder_16, origin xyz=0 0 0 rpy=0 0 0
- added joint j_baseToShoulder_17: type fixed, parent base_link, child baseToShoulder_17, origin xyz=0 0 0 rpy=0 0 0
- added joint j_baseToShoulder_18: type fixed, parent base_link, child baseToShoulder_18, origin xyz=0 0 0 rpy=0 0 0
- added joint j_baseToShoulder_19: type fixed, parent base_link, child baseToShoulder_19, origin xyz=0 0 0 rpy=0 0 0
- added joint j_baseToShoulder_20: type fixed, parent base_link, child baseToShoulder_20, origin xyz=0 0 0 rpy=0 0 0
- added joint j_baseToShoulder_21: type fixed, parent base_link, child baseToShoulder_21, origin xyz=0 0 0 rpy=0 0 0
- added joint j_baseToShoulder_22: type fixed, parent base_link, child baseToShoulder_22, origin xyz=0 0 0 rpy=0 0 0
- added joint j_baseToShoulder_23: type fixed, parent base_link, child baseToShoulder_23, origin xyz=0 0 0 rpy=0 0 0
- added joint j_baseToShoulder_24: type fixed, parent base_link, child baseToShoulder_24, origin xyz=0 0 0 rpy=0 0 0
- added joint j_baseToShoulder_25: type fixed, parent base_link, child baseToShoulder_25, origin xyz=0 0 0 rpy=0 0 0
- added joint j_baseToShoulder_26: type fixed, parent base_link, child baseToShoulder_26, origin xyz=0 0 0 rpy=0 0 0
- added joint j_baseToShoulder_27: type fixed, parent base_link, child baseToShoulder_27, origin xyz=0 0 0 rpy=0 0 0
- added joint j_baseToShoulder_28: type fixed, parent base_link, child baseToShoulder_28, origin xyz=0 0 0 rpy=0 0 0
- added joint j_baseToShoulder_29: type fixed, parent base_link, child baseToShoulder_29, origin xyz=0 0 0 rpy=0 0 0
- added joint j_baseToShoulder_30: type fixed, parent base_link, child baseToShoulder_30, origin xyz=0 0 0 rpy=0 0 0
- added joint j_baseToShoulder_31: type fixed, parent base_link, child baseToShoulder_31, origin xyz=0 0 0 rpy=0 0 0
- added joint j_baseToShoulder_32: type fixed, parent base_link, child baseToShoulder_32, origin xyz=0 0 0 rpy=0 0 0
- added joint j_carrier_to_pulley_01: type fixed, parent base_link, child carrier_to_pulley_01, origin xyz=0 0 0 rpy=0 0 0
- added joint j_carrier_to_pulley_02: type fixed, parent base_link, child carrier_to_pulley_02, origin xyz=0 0 0 rpy=0 0 0
- added joint j_carrier_to_pulley_03: type fixed, parent base_link, child carrier_to_pulley_03, origin xyz=0 0 0 rpy=0 0 0
- added joint j_carrier_to_pulley_04: type fixed, parent base_link, child carrier_to_pulley_04, origin xyz=0 0 0 rpy=0 0 0
- added joint j_carrier_to_pulley_05: type fixed, parent base_link, child carrier_to_pulley_05, origin xyz=0 0 0 rpy=0 0 0
- added joint j_full_arm_jun13_elbow: type fixed, parent base_link, child full_arm_jun13_elbow, origin xyz=0 0 0 rpy=0 0 0
- added joint j_key_to_diff_01: type fixed, parent base_link, child key_to_diff_01, origin xyz=0 0 0 rpy=0 0 0
- added joint j_key_to_diff_02: type fixed, parent base_link, child key_to_diff_02, origin xyz=0 0 0 rpy=0 0 0
- added joint j_key_to_diff_03: type fixed, parent base_link, child key_to_diff_03, origin xyz=0 0 0 rpy=0 0 0
- added joint j_key_to_diff_04: type fixed, parent base_link, child key_to_diff_04, origin xyz=0 0 0 rpy=0 0 0
- added joint j_key_to_diff_05: type fixed, parent base_link, child key_to_diff_05, origin xyz=0 0 0 rpy=0 0 0
- added joint j_key_to_diff_06: type fixed, parent base_link, child key_to_diff_06, origin xyz=0 0 0 rpy=0 0 0
- added joint j_key_to_diff_07: type fixed, parent base_link, child key_to_diff_07, origin xyz=0 0 0 rpy=0 0 0
- added joint j_key_to_diff_08: type fixed, parent base_link, child key_to_diff_08, origin xyz=0 0 0 rpy=0 0 0
- added joint j_key_to_diff_09: type fixed, parent base_link, child key_to_diff_09, origin xyz=0 0 0 rpy=0 0 0
- added joint j_key_to_diff_10: type fixed, parent base_link, child key_to_diff_10, origin xyz=0 0 0 rpy=0 0 0
- added joint j_key_to_diff_11: type fixed, parent base_link, child key_to_diff_11, origin xyz=0 0 0 rpy=0 0 0
- added joint j_key_to_diff_12: type fixed, parent base_link, child key_to_diff_12, origin xyz=0 0 0 rpy=0 0 0
- added joint world_to_base: type fixed, parent world, child base_link, origin xyz=0 0 0 rpy=0 0 0
