Commit message: Deleted the unused STL parts.

File: waybionic_description/urdf/full_arm_mar24.urdf (robot description, URDF)
Before this commit: robot full-arm-mar24-urdf-and-meshes, 5 links, 4 joints
Joints:
- joint joint1: axis 0 0 0 -> 0 0 1; type fixed -> revolute
- joint joint2: axis 0 0 0 -> 0 0 1; type fixed -> revolute
- joint joint4: axis 0 0 0 -> 0 0 1; limit (none) -> lower=-3.14 upper=3.14 effort=100 velocity=1; type fixed -> revolute

Commit message: Center arm model on RViz ground plane

File: waybionic_description/urdf/full_arm_mar24.urdf (robot description, URDF)
Before this commit: robot full-arm-mar24-urdf-and-meshes, 6 links, 5 joints
Joints:
- joint world_to_base: origin xyz=0 0 0 rpy=0 0 0 -> xyz=-0.800105 1.643392 -0.749746 rpy=0 0 0

Commit message: Polish and verify the IK demo

File: waybionic_description/urdf/full_arm_mar24.urdf (robot description, URDF)
Before this commit: robot full-arm-mar24-urdf-and-meshes, 6 links, 5 joints
Links:
- link base_link: geometry collision box size=0.54 0.47 0.51; collision cylinder length=0.070 radius=0.078
- link elbow: geometry collision box size=0.11 0.14 0.115; collision box size=0.11 0.34 0.17
- link forearm: geometry collision box size=0.09 0.17 0.12; collision box size=0.10 0.135 0.245
- link shoulder: geometry collision box size=0.21 0.235 0.14; collision cylinder length=0.070 radius=0.040
- link wrist: geometry collision box size=0.10 0.115 0.12; visual mesh filename=package://waybionic_description/meshes/wrist.STL

Commit message: Last commits before changes to new urdf

File: waybionic_description/urdf/full_arm_mar24.urdf (robot description, URDF)
Before this commit: robot full-arm-mar24-urdf-and-meshes, 6 links, 5 joints
Joints:
- joint joint1: limit lower=-3.14 upper=3.14 effort=100 velocity=1 -> lower=-1.5708 upper=1.5708 effort=100 velocity=1
- joint joint2: limit lower=-3.14 upper=3.14 effort=100 velocity=1 -> lower=-1.5708 upper=1.5708 effort=100 velocity=1
- joint joint3: limit lower=-3.14 upper=3.14 effort=100 velocity=1 -> lower=-1.5708 upper=1.5708 effort=100 velocity=1; type continuous -> revolute
- joint joint4: limit lower=-3.14 upper=3.14 effort=100 velocity=1 -> lower=-1.5708 upper=1.5708 effort=100 velocity=1

File: waybionic_moveit_config/urdf/waybionic_moveit.urdf.xacro (robot description, xacro)
@@ -17,6 +17,6 @@
     <joint name="joint1">
       <command_interface name="position">
-        <param name="min">-3.14</param>
-        <param name="max">3.14</param>
+        <param name="min">-1.5708</param>
+        <param name="max">1.5708</param>
       </command_interface>
       <state_interface name="position">
@@ -27,6 +27,6 @@
     <joint name="joint2">
       <command_interface name="position">
-        <param name="min">-3.14</param>
-        <param name="max">3.14</param>
+        <param name="min">-1.5708</param>
+        <param name="max">1.5708</param>
       </command_interface>
       <state_interface name="position">
@@ -35,7 +35,11 @@
       <state_interface name="velocity"/>
     </joint>
-    <!-- joint3 is a continuous joint: unbounded, so no min/max. -->
+    <!-- joint3 is now revolute (was continuous). Bounds must match the URDF
+         or the mock hardware accepts commands the model forbids. -->
     <joint name="joint3">
-      <command_interface name="position"/>
+      <command_interface name="position">
+        <param name="min">-1.5708</param>
+        <param name="max">1.5708</param>
+      </command_interface>
       <state_interface name="position">
         <param name="initial_value">0.0</param>
@@ -45,6 +49,6 @@
     <joint name="joint4">
       <command_interface name="position">
-        <param name="min">-3.14</param>
-        <param name="max">3.14</param>
+        <param name="min">-1.5708</param>
+        <param name="max">1.5708</param>
       </command_interface>
       <state_interface name="position">
