Commit message: Update joint limit upper value in URDF file
Co-authored-by: Copilot Autofix powered by AI <175728472+Copilot@users.noreply.github.com>

File: waybionic_description/urdf/old_arm_prototype.urdf (robot description, URDF)
Before this commit: robot waybionic_old_arm_prototype, 6 links, 5 joints
Joints:
- joint elbow: limit lower=-1.073377 upper=2.277655 effort=10 velocity=2.0 -> lower=-1.073377 upper=2.068215 effort=10 velocity=2.0
