Commit message: Add collision boxes and keep the arm off the table and its base
The URDF generator now writes a collision box around each link's mesh,
and the current URDF gets the boxes the generator would write.
ArmCollision reads the boxes and the joint tree from robot_description.
It reports any moving link that comes within the clearance of the table
plane, and any forearm or wrist part that comes within it of the base
or shoulder (separating axes).

Teleop undoes a step that would newly collide, in every group and when
going home, and lists the parts in blocked, so the diagnostics show for
example "forearm_link: table". A pose that already collides can still
move, so the arm can be backed out. Table height and clearance are in
xbox_teleop.yaml.

File: waybionic_description/urdf/waybionic_arm.urdf (robot description, URDF)
Before this commit: robot waybionic_arm, 9 links, 8 joints
Links:
- link base_link: geometry collision box size=0.2 0.2 0.1575; visual mesh filename=package://waybionic_description/meshes/arm/base_link.dae
- link forearm_link: geometry collision box size=0.096 0.144 0.3695; visual mesh filename=package://waybionic_description/meshes/arm/forearm_link.dae
- link shoulder_link: geometry collision box size=0.105 0.199 0.1405; visual mesh filename=package://waybionic_description/meshes/arm/shoulder_link.dae
- link upper_arm_link: geometry collision box size=0.105 0.175 0.26; visual mesh filename=package://waybionic_description/meshes/arm/upper_arm_link.d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
- link wrist_left_gear_link: geometry collision box size=0.053 0.0475 0.053; visual mesh filename=package://waybionic_description/meshes/arm/wrist_left_gear_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
- link wrist_pitch_link: geometry collision box size=0.08 0.082 0.083; visual mesh filename=package://waybionic_description/meshes/arm/wrist_pitch_link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
- link wrist_right_gear_link: geometry collision box size=0.053 0.0475 0.053; visual mesh filename=package://waybionic_description/meshes/arm/wrist_right_gear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
- link wrist_roll_link: geometry collision box size=0.07 0.0695 0.0815; visual mesh filename=package://waybionic_description/meshes/arm/wrist_roll_link.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

Commit message: Set joint limits where the CAD parts first touch
Each pitch joint stops 1 degree before two parts touch, found by scripts/cad/joint_clearance.py. Collision boxes follow each CAD part, and the elbow fold is checked against an exact table over the shoulder angle, kept in the URDF.

File: waybionic_description/urdf/waybionic_arm.urdf (robot description, URDF)
Before this commit: robot waybionic_arm, 9 links, 8 joints
Links:
- link base_link: geometry collision box size=0.0048 0.006 0.0228; collision box size=0.013 0.013 0.023
- link forearm_link: geometry collision box size=0.0144 0.0048 0.0048; collision box size=0.016 0.016 0.016
- link shoulder_link: geometry collision box size=0.02 0.037 0.021; collision box size=0.056 0.012 0.056
- link upper_arm_link: geometry collision box size=0.012 0.023 0.013; collision box size=0.048 0.0108 0.048
- link wrist_left_gear_link: geometry collision box size=0.0175 0.045 0.015; collision box size=0.04 0.016 0.04
- link wrist_right_gear_link: geometry collision box size=0.014 0.045 0.0165; collision box size=0.04 0.016 0.04
- link wrist_roll_link: geometry collision box size=0.06 0.06 0.049; collision box size=0.07 0.0695 0.0325
Joints:
- joint joint_2: limit lower=-1.570796 upper=1.570796 effort=0 velocity=0 -> lower=-2.356194 upper=2.356194 effort=0 velocity=0
- joint joint_3: limit lower=-1.570796 upper=1.570796 effort=0 velocity=0 -> lower=-2.565634 upper=2.565634 effort=0 velocity=0
- joint joint_4: limit lower=-1.570796 upper=1.570796 effort=0 velocity=0 -> lower=-1.623156 upper=1.623156 effort=0 velocity=0
- joint joint_5: limit lower=-1.570796 upper=1.570796 effort=0 velocity=0 -> lower=-3.141593 upper=3.141593 effort=0 velocity=0

Commit message: Keep the placeholder tool jaws clear with a collision box

File: waybionic_description/urdf/waybionic_arm.urdf (robot description, URDF)
Before this commit: robot waybionic_arm, 9 links, 8 joints
Links:
- link tool_link: geometry collision box size=0.036 0.014 0.03

Commit message: Align biomedical clamp collision and integration tests

File: waybionic_description/urdf/waybionic_arm.urdf (robot description, URDF)
Before this commit: robot waybionic_arm, 9 links, 8 joints
Links:
- link tool_link: geometry collision box size=0.08 0.08 0.1525

Commit message: Stop the arm where its CAD parts meet the base
The forearm now folds over the round base by a table of elbow limits
measured from the CAD at any yaw (joint_clearance.py, 2.5 degree steps),
as it already did against the shoulder. The build script gives a part
that is round about a joint axis a cylinder, and a part round on one
side, such as the wrist's differential housing, a cylinder with a box
for the rest, so the shapes fit those parts however the joints turn.
The collision check counts a cylinder as a 32-sided prism turned to
face the other shape, so spinning a round part about its own axis
cannot change a contact.

File: waybionic_description/urdf/waybionic_arm.urdf (robot description, URDF)
Before this commit: robot waybionic_arm, 9 links, 8 joints
Links:
- link base_link: geometry collision box size=0.0048 0.006 0.0228; collision box size=0.018 0.018 0.004
- link forearm_link: geometry collision box size=0.0144 0.0048 0.0048; collision box size=0.016 0.016 0.016
- link shoulder_link: geometry collision box size=0.056 0.103 0.068; collision box size=0.0636 0.0072 0.0636
- link upper_arm_link: geometry collision box size=0.048 0.0108 0.048; collision box size=0.048 0.0635 0.042
- link wrist_left_gear_link: geometry collision box size=0.0035 0.045 0.008; collision cylinder length=0.016 radius=0.0203
- link wrist_pitch_link: geometry collision box size=0.06 0.082 0.015; collision cylinder length=0.082 radius=0.04026
- link wrist_right_gear_link: geometry collision box size=0.01229 0.045 0.0045; collision cylinder length=0.016 radius=0.02016
- link wrist_roll_link: geometry collision cylinder length=0.0325 radius=0.03523; collision cylinder length=0.049 radius=0.03021

Commit message: Replace old wrist holder with biomedical clamp mount

File: waybionic_description/urdf/waybionic_arm.urdf (robot description, URDF)
Before this commit: robot waybionic_arm, 9 links, 8 joints
Links:
- link wrist_roll_link: geometry collision box size=0.06 0.06 0.049; visual mesh filename=package://waybionic_description/meshes/arm/wrist_roll_link.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
Joints:
- joint tool_joint: origin xyz=0 0 0.093369 rpy=0 0 0 -> xyz=0 0 0.061 rpy=0 0 0

Commit message: Set the joint limits where the CAD parts touch or meet the ground
scripts/cad/exact_limits.py turns each joint from the upright pose with exact triangle-mesh distances (FCL). The straight arm meets the ground under the base at 109.65 degrees of shoulder, the forearm meets the shoulder's motor mount at 148.93 degrees of elbow, and the tool mount meets the forearm's cap at 94.68 degrees of wrist pitch. Base yaw and wrist roll meet nothing over a full turn, so they turn 360 degrees either way. The elbow's fold tables now run to contact over the new shoulder range.

Against the table, the teleop check now uses each moving link's convex hull from the CAD (waybionic_hull in the URDF) instead of its collision shapes, which reached up to 12 mm below the tool mount. The table and self-collision clearances default to 0, so the arm stops where its parts touch.

File: waybionic_description/urdf/waybionic_arm.urdf (robot description, URDF)
Before this commit: robot waybionic_arm, 9 links, 8 joints
Joints:
- joint joint_1: limit lower=-3.141593 upper=3.141593 effort=0 velocity=0 -> lower=-6.283185 upper=6.283185 effort=0 velocity=0
- joint joint_2: limit lower=-2.356194 upper=2.356194 effort=0 velocity=0 -> lower=-1.913754 upper=1.913754 effort=0 velocity=0
- joint joint_3: limit lower=-2.565634 upper=2.565634 effort=0 velocity=0 -> lower=-2.599319 upper=2.599319 effort=0 velocity=0
- joint joint_4: limit lower=-1.623156 upper=1.623156 effort=0 velocity=0 -> lower=-1.652478 upper=1.652478 effort=0 velocity=0
- joint joint_5: limit lower=-3.141593 upper=3.141593 effort=0 velocity=0 -> lower=-6.283185 upper=6.283185 effort=0 velocity=0

Commit message: Stop the joint sliders where the arm's parts would touch
The sliders now go through joint_state_guard, which moves the arm toward the requested
pose with the teleop collision check, stops at the last pose before any part touches, and
sends the sliders back there. The wrist limit is now the lowest contact over a full turn of
roll (94.67 degrees), and scripts/cad/check_collision_model.py checks the collision model
against the CAD meshes.

File: waybionic_description/urdf/waybionic_arm.urdf (robot description, URDF)
Before this commit: robot waybionic_arm, 9 links, 8 joints
Joints:
- joint joint_4: limit lower=-1.652478 upper=1.652478 effort=0 velocity=0 -> lower=-1.652303 upper=1.652303 effort=0 velocity=0
